File: kicad/USBKB/USBKB.kicad_sch (KiCad schematic)
At the start: 69 parts, among them U1 ATMEGA32U4, U10 KAILH_CPG151101S11, U11 KAILH_CPG151101S11, U12 KAILH_CPG151101S11, U13 KAILH_CPG151101S11, U14 KAILH_CPG151101S11, U15 KAILH_CPG151101S11, U16 KAILH_CPG151101S11, U17 KAILH_CPG151101S11, U18 KAILH_CPG151101S11, U19 KAILH_CPG151101S11, U2 KAILH_CPG151101S11, U20 KAILH_CPG151101S11, U21 KAILH_CPG151101S11, U22 KAILH_CPG151101S11, U23 KAILH_CPG151101S11, U24 KAILH_CPG151101S11, U25 KAILH_CPG151101S11, U26 KAILH_CPG151101S11, U27 KAILH_CPG151101S11, U28 KAILH_CPG151101S11, U29 KAILH_CPG151101S11, U3 KAILH_CPG151101S11, U30 KAILH_CPG151101S11, U31 KAILH_CPG151101S11, U32 KAILH_CPG151101S11, U33 KAILH_CPG151101S11, U34 KAILH_CPG151101S11, U35 KAILH_CPG151101S11, U36 KAILH_CPG151101S11, U37 KAILH_CPG151101S11, U38 KAILH_CPG151101S11, U39 KAILH_CPG151101S11, U4 KAILH_CPG151101S11, U40 KAILH_CPG151101S11, U41 KAILH_CPG151101S11, U42 KAILH_CPG151101S11, U43 KAILH_CPG151101S11, U44 KAILH_CPG151101S11, U45 KAILH_CPG151101S11, U46 KAILH_CPG151101S11, U47 KAILH_CPG151101S11, U48 KAILH_CPG151101S11, U49 KAILH_CPG151101S11, U5 KAILH_CPG151101S11, U50 KAILH_CPG151101S11, U51 KAILH_CPG151101S11, U52 KAILH_CPG151101S11, U53 KAILH_CPG151101S11, U54 KAILH_CPG151101S11, U55 KAILH_CPG151101S11, U56 KAILH_CPG151101S11, U57 KAILH_CPG151101S11, U58 KAILH_CPG151101S11, U59 KAILH_CPG151101S11, U6 KAILH_CPG151101S11, U60 KAILH_CPG151101S11, U61 KAILH_CPG151101S11, U62 KAILH_CPG151101S11, U63 KAILH_CPG151101S11, U64 KAILH_CPG151101S11, U65 KAILH_CPG151101S11, U66 KAILH_CPG151101S11, U67 KAILH_CPG151101S11, U68 KAILH_CPG151101S11, U69 KAILH_CPG151101S11, U7 KAILH_CPG151101S11, U8 KAILH_CPG151101S11, U9 KAILH_CPG151101S11

Commit message: Work on PCB footprints
Parts:
- added C1: 1uF, symbol Device:C
- added R1, R2: 22, Resistor_SMD:R_0201_0603Metric, symbol Device:R
- added U70: UJ31-CH-G2-SMT-TR, symbol USBKB:UJ31-CH-G2-SMT-TR
- added U?: ICSP, symbol USBKB:ICSP
- U1: value ATMEGA32U4 -> ATMEGA32U4-MU; footprint USBKB:ATMEGA32U4 -> USBKB:ATMEGA32U4-MU; symbol USBKB:ATMEGA32U4 -> USBKB:ATMEGA32U4-MU
Connections:
- net +5V is gone; now on an unnamed net: U1.14 (Vcc), U1.24 (AVcc), U1.34 (Vcc), U1.42 (AREF), U1.44 (AVcc)
- net GND is gone; now on an unnamed net: U1.15 (GND), U1.23 (GND), U1.35 (GND), U1.43 (GND)
- net ROW1: now also U?.3 (SCK)
- net ROW2: now also U?.4 (MOSI)
- net ROW3: now also U?.1 (MISO)
- net at U1.13 (~{RESET}): now also U?.5 (RST)
- net at U1.2 (UVcc): now also U1.5 (UGnd), U1.7 (VBus), C1.1, U70.B1 (GND), U70.B12 (GND), U70.B4 (VBUS), U70.B9 (VBUS), U?.2 (Vcc), U?.6 (GND)
- net at U1.3 (D-): now also R2.1
- net at U1.4 (D+): now also R1.1
- net at U1.6 (UCap): now also C1.2
- new net: R2.2, U70.B7 (D-)
- new net: R1.2, U70.B6 (D+)
- no-connect marks 9 -> 14
Other:
- moved on the sheet: U10, U11, U12, U13, U14, U15, U16, U17, U18, U19, U2, U20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
