File: kicad/USBKB/USBKB.kicad_pcb (KiCad board)
At the start: 2 copper layers, 69 parts, among them U1 ATMEGA32U4, U10 KAILH_CPG151101S11, U11 KAILH_CPG151101S11, U12 KAILH_CPG151101S11, U13 KAILH_CPG151101S11, U14 KAILH_CPG151101S11, U15 KAILH_CPG151101S11, U16 KAILH_CPG151101S11, U17 KAILH_CPG151101S11, U18 KAILH_CPG151101S11, U19 KAILH_CPG151101S11, U2 KAILH_CPG151101S11, U20 KAILH_CPG151101S11, U21 KAILH_CPG151101S11, U22 KAILH_CPG151101S11, U23 KAILH_CPG151101S11, U24 KAILH_CPG151101S11, U25 KAILH_CPG151101S11, U26 KAILH_CPG151101S11, U27 KAILH_CPG151101S11, U28 KAILH_CPG151101S11, U29 KAILH_CPG151101S11, U3 KAILH_CPG151101S11, U30 KAILH_CPG151101S11, U31 KAILH_CPG151101S11, U32 KAILH_CPG151101S11, U33 KAILH_CPG151101S11, U34 KAILH_CPG151101S11, U35 KAILH_CPG151101S11, U36 KAILH_CPG151101S11, U37 KAILH_CPG151101S11, U38 KAILH_CPG151101S11, U39 KAILH_CPG151101S11, U4 KAILH_CPG151101S11, U40 KAILH_CPG151101S11, U41 KAILH_CPG151101S11, U42 KAILH_CPG151101S11, U43 KAILH_CPG151101S11, U44 KAILH_CPG151101S11, U45 KAILH_CPG151101S11, U46 KAILH_CPG151101S11, U47 KAILH_CPG151101S11, U48 KAILH_CPG151101S11, U49 KAILH_CPG151101S11, U5 KAILH_CPG151101S11, U50 KAILH_CPG151101S11, U51 KAILH_CPG151101S11, U52 KAILH_CPG151101S11, U53 KAILH_CPG151101S11, U54 KAILH_CPG151101S11, U55 KAILH_CPG151101S11, U56 KAILH_CPG151101S11, U57 KAILH_CPG151101S11, U58 KAILH_CPG151101S11, U59 KAILH_CPG151101S11, U6 KAILH_CPG151101S11, U60 KAILH_CPG151101S11, U61 KAILH_CPG151101S11, U62 KAILH_CPG151101S11, U63 KAILH_CPG151101S11, U64 KAILH_CPG151101S11, U65 KAILH_CPG151101S11, U66 KAILH_CPG151101S11, U67 KAILH_CPG151101S11, U68 KAILH_CPG151101S11, U69 KAILH_CPG151101S11, U7 KAILH_CPG151101S11, U8 KAILH_CPG151101S11, U9 KAILH_CPG151101S11

Commit message: Work on PCB footprints
Connections:
- U1 pad 14: +5V -> Net-(U1-Pad14)
- U1 pad 15: GND -> Net-(U1-Pad15)
- U1 pad 2: unconnected-(U1-Pad2) -> Net-(U1-Pad14)
- U1 pad 23: GND -> Net-(U1-Pad15)
- U1 pad 24: +5V -> Net-(U1-Pad14)
- U1 pad 3: unconnected-(U1-Pad3) -> Net-(U1-Pad3)
- U1 pad 34: +5V -> Net-(U1-Pad14)
- U1 pad 35: GND -> Net-(U1-Pad15)
- U1 pad 4: unconnected-(U1-Pad4) -> Net-(U1-Pad4)
- U1 pad 42: +5V -> Net-(U1-Pad14)
- U1 pad 43: GND -> Net-(U1-Pad15)
- U1 pad 44: +5V -> Net-(U1-Pad14)
- U1 pad 5: unconnected-(U1-Pad5) -> Net-(U1-Pad15)
- U1 pad 6: unconnected-(U1-Pad6) -> Net-(U1-Pad6)
- U1 pad 7: unconnected-(U1-Pad7) -> Net-(U1-Pad14)
Routing:
- net /COL6: track 77.3 -> 621.6 mm, vias 4 -> 0
- net /COL4: track 77.3 -> 612.3 mm, vias 4 -> 0
- net /COL5: track 0.00 -> 307.5 mm
- net /ROW4: track 307.5 -> 103.7 mm, vias 0 -> 5
- net /ROW2: track 305.7 -> 154.5 mm, vias 0 -> 8
- net /COL1: track 105.8 -> 0.00 mm, vias 5 -> 0
- net /COL12: track 105.7 -> 0.00 mm, vias 5 -> 0
- net /COL13: track 105.6 -> 0.00 mm, vias 5 -> 0
- net /COL11: track 104.5 -> 0.00 mm, vias 6 -> 0
- net /COL10: track 103.8 -> 0.00 mm, vias 6 -> 0
- net /COL2: track 103.7 -> 0.00 mm, vias 5 -> 0
- net /COL9: track 102.5 -> 0.00 mm, vias 5 -> 0
- net /COL8: track 99.6 -> 0.00 mm, vias 5 -> 0
- net /COL0: track 98.0 -> 0.00 mm, vias 5 -> 0
- net /ROW3: track 302.4 -> 389.8 mm, vias 0 -> 20
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
Commit message: Schematic and footprint complete
Parts:
- removed U1: ATMEGA32U4, USBKB:ATMEGA32U4
- removed U10, U11, U12, U13, U14, U15, U16, U17, U18, U19, U2, U20, U21, U22, U23, U24, U25, U26, U27, U28, U29, U3, U30, U31, U32, U33, U34, U35, U36, U37, U38, U39, U4, U40, U41, U42, U43, U44, U45, U46, U47, U48, U49, U5, U50, U51, U52, U53, U54, U55, U56, U57, U58, U59, U6, U60, U61, U62, U63, U64, U65, U66, U67, U68, U69, U7, U8, U9: KAILH_CPG151101S11, USBKB:KAILH CPG151101S11
Routing:
- net /COL6: track 621.6 -> 0.00 mm
- net /COL4: track 612.3 -> 0.00 mm
- net /ROW3: track 389.8 -> 0.00 mm, vias 20 -> 0
- net /ROW0: track 333.8 -> 0.00 mm, vias 18 -> 0
- net /COL5: track 307.5 -> 0.00 mm
- net /ROW1: track 281.1 -> 0.00 mm, vias 14 -> 0
- net /ROW2: track 154.5 -> 0.00 mm, vias 8 -> 0
- net /ROW4: track 103.7 -> 0.00 mm, vias 5 -> 0

Commit message: Began PCB alignment
Parts:
- added C1: 1uF, USBKB:0805, F.Cu at (118.0, 103.0)
- added C2: 22pF, USBKB:0805, F.Cu at (122.0, 107.0)
- added C3: 22pF, USBKB:0805, F.Cu at (112.0, 104.0)
- added KA1: KAILH_CPG151101S11, USBKB:KAILH-CPG151101S11-1U, F.Cu at (60.6, 65.0)
- added KAP1: KAILH_CPG151101S11, USBKB:KAILH-CPG151101S11-1U, F.Cu at (251.1, 65.0)
- added KB1: KAILH_CPG151101S11, USBKB:KAILH-CPG151101S11-1U, F.Cu at (146.3, 84.1)
- added KBSLASH1: KAILH_CPG151101S11, USBKB:KAILH-CPG151101S11-1.5U, F.Cu at (289.2, 46.0)
- added KBSPACE1: KAILH_CPG151101S11, USBKB:KAILH-CPG151101S11-2U, F.Cu at (284.5, 26.9)
- added KC1: KAILH_CPG151101S11, USBKB:KAILH-CPG151101S11-1U, F.Cu at (108.2, 84.1)
- added KCAPS1: KAILH_CPG151101S11, USBKB:KAILH-CPG151101S11-1.75U, F.Cu at (34.4, 65.0)
- added KCOMMA1: KAILH_CPG151101S11, USBKB:KAILH-CPG151101S11-1U, F.Cu at (203.5, 84.1)
- added KD1: KAILH_CPG151101S11, USBKB:KAILH-CPG151101S11-1U, F.Cu at (98.7, 65.0)
- added KDASH1: KAILH_CPG151101S11, USBKB:KAILH-CPG151101S11-1U, F.Cu at (236.8, 26.9)
- added KE1: KAILH_CPG151101S11, USBKB:KAILH-CPG151101S11-1U, F.Cu at (94.0, 46.0)
- added KEIGHT1: KAILH_CPG151101S11, USBKB:KAILH-CPG151101S11-1U, F.Cu at (179.7, 26.9)
- added KEQUALS1: KAILH_CPG151101S11, USBKB:KAILH-CPG151101S11-1U, F.Cu at (255.9, 26.9)
- added KESC1: KAILH_CPG151101S11, USBKB:KAILH-CPG151101S11-1U, F.Cu at (27.3, 26.9)
- added KF1: KAILH_CPG151101S11, USBKB:KAILH-CPG151101S11-1U, F.Cu at (117.8, 65.0)
- added KFIVE1: KAILH_CPG151101S11, USBKB:KAILH-CPG151101S11-1U, F.Cu at (122.5, 26.9)
- added KFN1: KAILH_CPG151101S11, USBKB:KAILH-CPG151101S11-1.25U, F.Cu at (291.6, 103.2)
- added KFOUR1: KAILH_CPG151101S11, USBKB:KAILH-CPG151101S11-1U, F.Cu at (103.5, 26.9)
- added KFSLASH1: KAILH_CPG151101S11, USBKB:KAILH-CPG151101S11-1U, F.Cu at (241.6, 84.1)
- added KG1: KAILH_CPG151101S11, USBKB:KAILH-CPG151101S11-1U, F.Cu at (136.8, 65.0)
- added KH1: KAILH_CPG151101S11, USBKB:KAILH-CPG151101S11-1U, F.Cu at (155.9, 65.0)
- added KI1: KAILH_CPG151101S11, USBKB:KAILH-CPG151101S11-1U, F.Cu at (189.2, 46.0)
- added KJ1: KAILH_CPG151101S11, USBKB:KAILH-CPG151101S11-1U, F.Cu at (174.9, 65.0)
- added KK1: KAILH_CPG151101S11, USBKB:KAILH-CPG151101S11-1U, F.Cu at (194.0, 65.0)
- added KL1: KAILH_CPG151101S11, USBKB:KAILH-CPG151101S11-1U, F.Cu at (213.0, 65.0)
- added KLALT1: KAILH_CPG151101S11, USBKB:KAILH-CPG151101S11-1.25U, F.Cu at (77.3, 103.2)
- added KLB1: KAILH_CPG151101S11, USBKB:KAILH-CPG151101S11-1U, F.Cu at (246.3, 46.0)
- added KLCTRL1: KAILH_CPG151101S11, USBKB:KAILH-CPG151101S11-1.25U, F.Cu at (29.7, 103.2)
- added KLMETA1: KAILH_CPG151101S11, USBKB:KAILH-CPG151101S11-1.25U, F.Cu at (53.5, 103.2)
- added KLS1: KAILH_CPG151101S11, USBKB:KAILH-CPG151101S11-2.25U, F.Cu at (39.2, 84.1)
- added KM1: KAILH_CPG151101S11, USBKB:KAILH-CPG151101S11-1U, F.Cu at (184.4, 84.1)
- added KN1: KAILH_CPG151101S11, USBKB:KAILH-CPG151101S11-1U, F.Cu at (165.4, 84.1)
- added KNINE1: KAILH_CPG151101S11, USBKB:KAILH-CPG151101S11-1U, F.Cu at (198.7, 26.9)
- added KO1: KAILH_CPG151101S11, USBKB:KAILH-CPG151101S11-1U, F.Cu at (208.2, 46.0)
- added KONE1: KAILH_CPG151101S11, USBKB:KAILH-CPG151101S11-1U, F.Cu at (46.3, 26.9)
- added KP1: KAILH_CPG151101S11, USBKB:KAILH-CPG151101S11-1U, F.Cu at (227.3, 46.0)
- added KPERIOD1: KAILH_CPG151101S11, USBKB:KAILH-CPG151101S11-1U, F.Cu at (222.5, 84.1)
- added KQ1: KAILH_CPG151101S11, USBKB:KAILH-CPG151101S11-1U, F.Cu at (55.9, 46.0)
- added KR1: KAILH_CPG151101S11, USBKB:KAILH-CPG151101S11-1U, F.Cu at (113.0, 46.0)
- added KRALT1: KAILH_CPG151101S11, USBKB:KAILH-CPG151101S11-1.25U, F.Cu at (220.2, 103.2)
- added KRB1: KAILH_CPG151101S11, USBKB:KAILH-CPG151101S11-1U, F.Cu at (265.4, 46.0)
- added KRCTRL1: KAILH_CPG151101S11, USBKB:KAILH-CPG151101S11-1.25U, F.Cu at (267.8, 103.2)
- added KRETURN1: KAILH_CPG151101S11, USBKB:KAILH-CPG151101S11-2.25U, F.Cu at (282.1, 65.0)
- added KRMETA1: KAILH_CPG151101S11, USBKB:KAILH-CPG151101S11-1.25U, F.Cu at (244.0, 103.2)
- added KRS1: KAILH_CPG151101S11, USBKB:KAILH-CPG151101S11-2.75U, F.Cu at (277.3, 84.1)
- added KS1: KAILH_CPG151101S11, USBKB:KAILH-CPG151101S11-1U, F.Cu at (79.7, 65.0)
- added KSC1: KAILH_CPG151101S11, USBKB:KAILH-CPG151101S11-1U, F.Cu at (232.1, 65.0)
- added KSEVEN1: KAILH_CPG151101S11, USBKB:KAILH-CPG151101S11-1U, F.Cu at (160.6, 26.9)
- added KSIX1: KAILH_CPG151101S11, USBKB:KAILH-CPG151101S11-1U, F.Cu at (141.6, 26.9)
- added KSPACE1: KAILH_CPG151101S11, USBKB:KAILH-CPG151101S11-6.25U, F.Cu at (148.7, 103.2)
- added KT1: KAILH_CPG151101S11, USBKB:KAILH-CPG151101S11-1U, F.Cu at (132.0, 46.0)
- added KTAB1: KAILH_CPG151101S11, USBKB:KAILH-CPG151101S11-1.5U, F.Cu at (32.0, 46.0)
- added KTHREE1: KAILH_CPG151101S11, USBKB:KAILH-CPG151101S11-1U, F.Cu at (84.4, 26.9)
- added KTWO1: KAILH_CPG151101S11, USBKB:KAILH-CPG151101S11-1U, F.Cu at (65.4, 26.9)
- added KU1: KAILH_CPG151101S11, USBKB:KAILH-CPG151101S11-1U, F.Cu at (170.1, 46.0)
- added KV1: KAILH_CPG151101S11, USBKB:KAILH-CPG151101S11-1U, F.Cu at (127.3, 84.1)
- added KW1: KAILH_CPG151101S11, USBKB:KAILH-CPG151101S11-1U, F.Cu at (74.9, 46.0)
- added KX1: KAILH_CPG151101S11, USBKB:KAILH-CPG151101S11-1U, F.Cu at (89.2, 84.1)
- added KY1: KAILH_CPG151101S11, USBKB:KAILH-CPG151101S11-1U, F.Cu at (151.1, 46.0)
- added KZ1: KAILH_CPG151101S11, USBKB:KAILH-CPG151101S11-1U, F.Cu at (70.1, 84.1)
- added KZERO1: KAILH_CPG151101S11, USBKB:KAILH-CPG151101S11-1U, F.Cu at (217.8, 26.9)
- added R1: 22, USBKB:0805, F.Cu at (130.0, 104.0)
- added R2: 22, USBKB:0805, F.Cu at (109.0, 109.0)
- added U1: USB4105-GF-A, USBKB:USB4105-GF-A, F.Cu at (35.0, 14.4)
- added U2: ICSP, USBKB:ICSP, F.Cu at (200.0, 103.0)
- added U3: ATMEGA32U4-MU, USBKB:ATMEGA32U4-MU, F.Cu at (176.0, 101.0)
- added Y1: Crystal_GND23, USBKB:ABM8G, F.Cu at (163.0, 103.0)

Commit message: Plate and PCB completed, pricing list updated with shipping fees
Parts:
- C1, C2, C3, R1, R2, U3, Y1: moved to B.Cu
- moved U3 61.8 mm to (115.5, 113.5), turned to 180 degrees
- moved Y1 33.4 mm to (134.5, 120.5), turned to 180 degrees
- moved C3 30.5 mm to (140.0, 116.0)
- moved U2 25.7 mm to (177.0, 114.5)
- moved C2 21.9 mm to (140.0, 119.5)
- moved C1 19.5 mm to (133.5, 114.8)
- moved R2 18.8 mm to (127.8, 109.0), turned to 180 degrees
- moved U1 14.4 mm to (40.9, 27.5)
- moved KAP1 13.4 mm to (257.0, 77.0)
- moved KBSLASH1 13.4 mm to (295.1, 58.0)
- moved KFN1 13.4 mm to (297.5, 115.2)
- moved KRB1 13.4 mm to (271.3, 58.0)
- moved KA1 13.4 mm to (66.5, 77.0)
- moved KESC1 13.4 mm to (33.2, 39.0)
- moved KDASH1 13.4 mm to (242.7, 39.0)
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Connections:
- C3 pad 2: Net-(Y1-Pad4) -> Net-(C3-Pad2)
- U1 pad A4/B9: Net-(C1-Pad1) -> Net-(U1-PadA4/B9)
- U1 pad B4/A9: Net-(C1-Pad1) -> Net-(U1-PadA4/B9)
- U2 pad 1: /ROW3 -> /ROW1
- U2 pad 2: Net-(C1-Pad1) -> Net-(U1-PadA4/B9)
- U2 pad 3: /ROW1 -> /ROW3
- U3 pad 11: /ROW3 -> /ROW1
- U3 pad 12: /COL2 -> /ROW0
- U3 pad 14: Net-(C1-Pad1) -> Net-(U1-PadA4/B9)
- U3 pad 16: Net-(Y1-Pad4) -> Net-(C3-Pad2)
- U3 pad 18: /COL3 -> /COL0
- U3 pad 19: /COL4 -> /COL1
- U3 pad 2: Net-(C1-Pad1) -> Net-(U1-PadA4/B9)
- U3 pad 20: /COL5 -> /COL2
- U3 pad 21: /COL6 -> /COL3
- U3 pad 22: /COL7 -> /COL4
- U3 pad 24: Net-(C1-Pad1) -> Net-(U1-PadA4/B9)
- U3 pad 25: /COL8 -> /COL5
- U3 pad 26: /COL9 -> /COL6
- U3 pad 27: /COL10 -> /COL7
- U3 pad 28: /ROW4 -> /COL8
- U3 pad 29: /COL0 -> /COL9
- U3 pad 30: /COL1 -> /COL10
- U3 pad 31: unconnected-(U3-Pad31) -> /COL11
- U3 pad 32: unconnected-(U3-Pad32) -> /COL12
- U3 pad 33: unconnected-(U3-Pad33) -> /COL13
- U3 pad 34: Net-(C1-Pad1) -> Net-(U1-PadA4/B9)
- U3 pad 39: /COL13 -> unconnected-(U3-Pad39)
- U3 pad 40: /COL12 -> unconnected-(U3-Pad40)
- U3 pad 41: /COL11 -> unconnected-(U3-Pad41)
- U3 pad 42: Net-(C1-Pad1) -> Net-(U1-PadA4/B9)
- U3 pad 44: Net-(C1-Pad1) -> Net-(U1-PadA4/B9)
- U3 pad 7: Net-(C1-Pad1) -> Net-(U1-PadA4/B9)
- U3 pad 8: /ROW0 -> /ROW4
- U3 pad 9: /ROW1 -> /ROW3
- Y1 pad 3: Net-(C1-Pad1) -> Net-(C3-Pad2)
- Y1 pad 4: Net-(Y1-Pad4) -> Net-(C1-Pad1)
Routing:
- net Net-(U1-PadA4/B9): track 0.00 -> 715.9 mm, vias 0 -> 7
- net Net-(C1-Pad1): track 0.00 -> 673.3 mm, vias 0 -> 2
- net /ROW1: track 0.00 -> 663.0 mm, vias 0 -> 4
- net /ROW2: track 0.00 -> 649.2 mm, vias 0 -> 2
- net /ROW0: track 0.00 -> 627.6 mm, vias 0 -> 2
- net /ROW3: track 0.00 -> 606.8 mm, vias 0 -> 4
- net Net-(R2-Pad2): track 0.00 -> 565.3 mm, vias 0 -> 3
- net Net-(R1-Pad2): track 0.00 -> 561.3 mm, vias 0 -> 1
- net /ROW4: track 0.00 -> 527.9 mm, vias 0 -> 4
- net /COL11: track 0.00 -> 298.6 mm, vias 0 -> 5
- net /COL12: track 0.00 -> 274.4 mm, vias 0 -> 4
- net /COL13: track 0.00 -> 267.8 mm, vias 0 -> 3
- net /COL10: track 0.00 -> 265.1 mm, vias 0 -> 5
- net /COL9: track 0.00 -> 242.4 mm, vias 0 -> 5
- net /COL8: track 0.00 -> 219.9 mm, vias 0 -> 5
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Other:
- board outline added: 289.8 x 105.6 mm
