File: design/pcb/USBKB.kicad_pcb (KiCad board)
At the start: 2 copper layers, 289.8 x 105.6 mm, 70 parts, among them U1 USB4105-GF-A, U2 ICSP, U3 ATMEGA32U4-MU, Y1 Crystal_GND23

Commit message: Work on case and PCB (now completely rectangular)
Parts:
- moved U1 5.90 mm to (40.8, 33.4)
- turned KESC1 to 180 degrees
- turned KONE1 to 180 degrees
Routing:
- net /ROW0: track 627.6 -> 652.1 mm
- net /COL1: track 173.2 -> 166.2 mm
- net /COL0: track 188.2 -> 193.2 mm
- net Net-(C1-Pad1): track 673.3 -> 677.9 mm, vias 2 -> 4
- net Net-(U1-PadA4/B9): track 715.9 -> 712.5 mm
- net Net-(R2-Pad2): track 565.3 -> 567.2 mm, vias 3 -> 1
- net Net-(R1-Pad2): track 561.3 -> 560.0 mm
Other:
- board size 289.8 x 105.6 mm -> 289.8 x 99.2 mm

Commit message: Changes to PCB layout, design, diodes, leds, code, everything
Parts:
- added DA1: D, USBKB:1N4148WX, B.Cu at (62.6, 66.6)
- added DAP1: D, USBKB:1N4148WX, B.Cu at (253.1, 66.6)
- added DB1: D, USBKB:1N4148WX, B.Cu at (148.3, 85.7)
- added DBSLASH1: D, USBKB:1N4148WX, B.Cu at (291.2, 47.6)
- added DBSPACE1: D, USBKB:1N4148WX, B.Cu at (286.4, 28.5)
- added DC1: D, USBKB:1N4148WX, B.Cu at (110.2, 85.7)
- added DCAPS1: D, USBKB:1N4148WX, B.Cu at (36.4, 66.6)
- added DCOMMA1: D, USBKB:1N4148WX, B.Cu at (205.5, 85.7)
- added DD1: D, USBKB:1N4148WX, B.Cu at (100.7, 66.6)
- added DDASH1: D, USBKB:1N4148WX, B.Cu at (238.8, 28.5)
- added DE1: D, USBKB:1N4148WX, B.Cu at (95.9, 47.6)
- added DEIGHT1: D, USBKB:1N4148WX, B.Cu at (181.7, 28.5)
- added DEQUALS1: D, USBKB:1N4148WX, B.Cu at (257.9, 28.5)
- added DESC1: D, USBKB:1N4148WX, B.Cu at (29.3, 28.5)
- added DF1: D, USBKB:1N4148WX, B.Cu at (119.8, 66.6)
- added DFIVE1: D, USBKB:1N4148WX, B.Cu at (124.5, 28.5)
- added DFN1: D, USBKB:1N4148WX, B.Cu at (293.6, 104.7)
- added DFOUR1: D, USBKB:1N4148WX, B.Cu at (105.5, 28.5)
- added DFSLASH1: D, USBKB:1N4148WX, B.Cu at (243.6, 85.7)
- added DG1: D, USBKB:1N4148WX, B.Cu at (138.8, 66.6)
- added DH1: D, USBKB:1N4148WX, B.Cu at (157.9, 66.6)
- added DI1: D, USBKB:1N4148WX, B.Cu at (191.2, 47.6)
- added DJ1: D, USBKB:1N4148WX, B.Cu at (176.9, 66.6)
- added DK1: D, USBKB:1N4148WX, B.Cu at (196.0, 66.6)
- added DL1: D, USBKB:1N4148WX, B.Cu at (215.0, 66.6)
- added DLALT1: D, USBKB:1N4148WX, B.Cu at (79.3, 104.7)
- added DLB1: D, USBKB:1N4148WX, B.Cu at (248.3, 47.6)
- added DLCTRL1: D, USBKB:1N4148WX, B.Cu at (31.7, 104.7)
- added DLMETA1: D, USBKB:1N4148WX, B.Cu at (55.5, 104.7)
- added DLS1: D, USBKB:1N4148WX, B.Cu at (41.2, 85.7)
- added DM1: D, USBKB:1N4148WX, B.Cu at (186.4, 85.7)
- added DN1: D, USBKB:1N4148WX, B.Cu at (167.4, 85.7)
- added DNINE1: D, USBKB:1N4148WX, B.Cu at (200.7, 28.5)
- added DO1: D, USBKB:1N4148WX, B.Cu at (210.2, 47.6)
- added DONE1: D, USBKB:1N4148WX, B.Cu at (48.3, 28.5)
- added DP1: D, USBKB:1N4148WX, B.Cu at (229.3, 47.6)
- added DPERIOD1: D, USBKB:1N4148WX, B.Cu at (224.5, 85.7)
- added DQ1: D, USBKB:1N4148WX, B.Cu at (57.8, 47.6)
- added DR1: D, USBKB:1N4148WX, B.Cu at (115.0, 47.6)
- added DRALT1: D, USBKB:1N4148WX, B.Cu at (222.2, 104.7)
- added DRB1: D, USBKB:1N4148WX, B.Cu at (267.4, 47.6)
- added DRCTRL1: D, USBKB:1N4148WX, B.Cu at (269.8, 104.7)
- added DRETURN1: D, USBKB:1N4148WX, B.Cu at (284.1, 66.6)
- added DRMETA1: D, USBKB:1N4148WX, B.Cu at (246.0, 104.7)
- added DRS1: D, USBKB:1N4148WX, B.Cu at (279.3, 85.7)
- added DS1: D, USBKB:1N4148WX, B.Cu at (81.7, 66.6)
- added DSC1: D, USBKB:1N4148WX, B.Cu at (234.1, 66.6)
- added DSEVEN1: D, USBKB:1N4148WX, B.Cu at (162.6, 28.5)
- added DSIX1: D, USBKB:1N4148WX, B.Cu at (143.6, 28.5)
- added DSPACE1: D, USBKB:1N4148WX, B.Cu at (150.7, 104.7)
- added DT1: D, USBKB:1N4148WX, B.Cu at (134.0, 47.6)
- added DTAB1: D, USBKB:1N4148WX, B.Cu at (34.0, 47.6)
- added DTHREE1: D, USBKB:1N4148WX, B.Cu at (86.4, 28.5)
- added DTWO1: D, USBKB:1N4148WX, B.Cu at (67.4, 28.5)
- added DU1: D, USBKB:1N4148WX, B.Cu at (172.1, 47.6)
- added DV1: D, USBKB:1N4148WX, B.Cu at (129.3, 85.7)
- added DW1: D, USBKB:1N4148WX, B.Cu at (76.9, 47.6)
- added DX1: D, USBKB:1N4148WX, B.Cu at (91.2, 85.7)
- added DY1: D, USBKB:1N4148WX, B.Cu at (153.1, 47.6)
- added DZ1: D, USBKB:1N4148WX, B.Cu at (72.1, 85.7)
- added DZERO1: D, USBKB:1N4148WX, B.Cu at (219.8, 28.5)
- added LA1: WS2812B, USBKB:SK6812MINI-E, B.Cu at (55.4, 55.6)
- added LAP1: WS2812B, USBKB:SK6812MINI-E, B.Cu at (245.9, 55.6)
- added LB1: WS2812B, USBKB:SK6812MINI-E, B.Cu at (141.1, 74.7)
- added LBSLASH1: WS2812B, USBKB:SK6812MINI-E, B.Cu at (284.0, 36.6)
- added LBSPACE1: WS2812B, USBKB:SK6812MINI-E, B.Cu at (279.2, 17.5)
- added LC1: WS2812B, USBKB:SK6812MINI-E, B.Cu at (103.0, 74.7)
- added LCAPS1: WS2812B, USBKB:SK6812MINI-E, B.Cu at (29.2, 55.6)
- added LCOMMA1: WS2812B, USBKB:SK6812MINI-E, B.Cu at (198.2, 74.7)
- added LD1: WS2812B, USBKB:SK6812MINI-E, B.Cu at (93.5, 55.6)
- added LDASH1: WS2812B, USBKB:SK6812MINI-E, B.Cu at (231.6, 17.5)
- added LE1: WS2812B, USBKB:SK6812MINI-E, B.Cu at (88.7, 36.6)
- added LEIGHT1: WS2812B, USBKB:SK6812MINI-E, B.Cu at (174.4, 17.5)
- added LEQUALS1: WS2812B, USBKB:SK6812MINI-E, B.Cu at (250.6, 17.5)
- added LESC1: WS2812B, USBKB:SK6812MINI-E, B.Cu at (22.0, 17.5)
- added LF1: WS2812B, USBKB:SK6812MINI-E, B.Cu at (112.5, 55.6)
- added LFIVE1: WS2812B, USBKB:SK6812MINI-E, B.Cu at (117.3, 17.5)
- added LFN1: WS2812B, USBKB:SK6812MINI-E, B.Cu at (286.3, 93.7)
- added LFOUR1: WS2812B, USBKB:SK6812MINI-E, B.Cu at (98.2, 17.5)
- added LFSLASH1: WS2812B, USBKB:SK6812MINI-E, B.Cu at (236.3, 74.7)
- added LG1: WS2812B, USBKB:SK6812MINI-E, B.Cu at (131.6, 55.6)
- added LH1: WS2812B, USBKB:SK6812MINI-E, B.Cu at (150.6, 55.6)
- added LI1: WS2812B, USBKB:SK6812MINI-E, B.Cu at (183.9, 36.6)
- added LJ1: WS2812B, USBKB:SK6812MINI-E, B.Cu at (169.7, 55.6)
- added LK1: WS2812B, USBKB:SK6812MINI-E, B.Cu at (188.7, 55.6)
- added LL1: WS2812B, USBKB:SK6812MINI-E, B.Cu at (207.8, 55.6)
- added LLALT1: WS2812B, USBKB:SK6812MINI-E, B.Cu at (72.0, 93.7)
- added LLB1: WS2812B, USBKB:SK6812MINI-E, B.Cu at (241.1, 36.6)
- added LLCTRL1: WS2812B, USBKB:SK6812MINI-E, B.Cu at (24.4, 93.7)
- added LLS1: WS2812B, USBKB:SK6812MINI-E, B.Cu at (33.9, 74.7)
- added LM1: WS2812B, USBKB:SK6812MINI-E, B.Cu at (179.2, 74.7)
- added LMETA1: WS2812B, USBKB:SK6812MINI-E, B.Cu at (48.2, 93.7)
- added LN1: WS2812B, USBKB:SK6812MINI-E, B.Cu at (160.1, 74.7)
- added LNINE1: WS2812B, USBKB:SK6812MINI-E, B.Cu at (193.5, 17.5)
- added LO1: WS2812B, USBKB:SK6812MINI-E, B.Cu at (203.0, 36.6)
- added LONE1: WS2812B, USBKB:SK6812MINI-E, B.Cu at (41.1, 17.5)
- added LP1: WS2812B, USBKB:SK6812MINI-E, B.Cu at (222.0, 36.6)
- added LPERIOD1: WS2812B, USBKB:SK6812MINI-E, B.Cu at (217.3, 74.7)
- added LQ1: WS2812B, USBKB:SK6812MINI-E, B.Cu at (50.6, 36.6)
- added LR1: WS2812B, USBKB:SK6812MINI-E, B.Cu at (107.7, 36.6)
- added LRALT1: WS2812B, USBKB:SK6812MINI-E, B.Cu at (214.9, 93.7)
- added LRB1: WS2812B, USBKB:SK6812MINI-E, B.Cu at (260.1, 36.6)
- added LRCTRL1: WS2812B, USBKB:SK6812MINI-E, B.Cu at (262.5, 93.7)
- added LRETURN1: WS2812B, USBKB:SK6812MINI-E, B.Cu at (276.8, 55.6)
- added LRMETA1: WS2812B, USBKB:SK6812MINI-E, B.Cu at (238.7, 93.7)
- added LRS1: WS2812B, USBKB:SK6812MINI-E, B.Cu at (272.1, 74.7)
- added LS1: WS2812B, USBKB:SK6812MINI-E, B.Cu at (74.4, 55.6)
- added LSC1: WS2812B, USBKB:SK6812MINI-E, B.Cu at (226.8, 55.6)
- added LSEVEN1: WS2812B, USBKB:SK6812MINI-E, B.Cu at (155.4, 17.5)
- added LSIX1: WS2812B, USBKB:SK6812MINI-E, B.Cu at (136.3, 17.5)
- added LSPACE1: WS2812B, USBKB:SK6812MINI-E, B.Cu at (143.5, 93.7)
- added LT1: WS2812B, USBKB:SK6812MINI-E, B.Cu at (126.8, 36.6)
- added LTAB1: WS2812B, USBKB:SK6812MINI-E, B.Cu at (26.8, 36.6)
- added LTHREE1: WS2812B, USBKB:SK6812MINI-E, B.Cu at (79.2, 17.5)
- added LTWO1: WS2812B, USBKB:SK6812MINI-E, B.Cu at (60.1, 17.5)
- added LU1: WS2812B, USBKB:SK6812MINI-E, B.Cu at (164.9, 36.6)
- added LV1: WS2812B, USBKB:SK6812MINI-E, B.Cu at (122.0, 74.7)
- added LW1: WS2812B, USBKB:SK6812MINI-E, B.Cu at (69.6, 36.6)
- added LX1: WS2812B, USBKB:SK6812MINI-E, B.Cu at (83.9, 74.7)
- added LY1: WS2812B, USBKB:SK6812MINI-E, B.Cu at (145.8, 36.6)
- added LZ1: WS2812B, USBKB:SK6812MINI-E, B.Cu at (64.9, 74.7)
- added LZERO1: WS2812B, USBKB:SK6812MINI-E, B.Cu at (212.5, 17.5)
- U1: moved to B.Cu
- moved KRB1 20.3 mm to (260.1, 41.1), turned to 180 degrees
- moved KLALT1 20.3 mm to (72.0, 98.2), turned to 180 degrees
- moved KAP1 20.3 mm to (245.9, 60.1), turned to 180 degrees
- moved KLB1 20.3 mm to (241.1, 41.1), turned to 180 degrees
- moved KO1 20.3 mm to (203.0, 41.1), turned to 180 degrees
- moved KU1 20.3 mm to (164.9, 41.1), turned to 180 degrees
- moved KESC1 20.3 mm to (22.0, 22.0)
- moved KFN1 20.3 mm to (286.3, 98.2), turned to 180 degrees
- moved KLCTRL1 20.3 mm to (24.4, 98.2), turned to 180 degrees
- moved KLMETA1 20.3 mm to (48.2, 98.2), turned to 180 degrees
- moved KONE1 20.3 mm to (41.1, 22.0)
- moved KRALT1 20.3 mm to (214.9, 98.2), turned to 180 degrees
- moved KRCTRL1 20.3 mm to (262.5, 98.2), turned to 180 degrees
- moved KRMETA1 20.3 mm to (238.7, 98.2), turned to 180 degrees
- moved KSPACE1 20.3 mm to (143.5, 98.2), turned to 180 degrees
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- renumbered U3 to M1
Connections:
- net Net-(U1-PadA4/B9) renamed VCC
- C1 pad 1: Net-(C1-Pad1) -> GND
- C2 pad 1: Net-(C1-Pad1) -> GND
- C3 pad 1: Net-(C1-Pad1) -> Net-(C3-Pad1)
- C3 pad 2: Net-(C3-Pad2) -> GND
- KA1 pad 2: /COL1 -> Net-(DA1-Pad2)
- KAP1 pad 2: /COL11 -> Net-(DAP1-Pad2)
- KB1 pad 2: /COL5 -> Net-(DB1-Pad2)
- KBSLASH1 pad 2: /COL13 -> Net-(DBSLASH1-Pad2)
- KBSPACE1 pad 2: /COL13 -> Net-(DBSPACE1-Pad2)
- KC1 pad 2: /COL3 -> Net-(DC1-Pad2)
- KCAPS1 pad 2: /COL0 -> Net-(DCAPS1-Pad2)
- KCOMMA1 pad 2: /COL8 -> Net-(DCOMMA1-Pad2)
- KD1 pad 2: /COL3 -> Net-(DD1-Pad2)
- KDASH1 pad 2: /COL11 -> Net-(DDASH1-Pad2)
- KE1 pad 2: /COL3 -> Net-(DE1-Pad2)
- KEIGHT1 pad 2: /COL8 -> Net-(DEIGHT1-Pad2)
- KEQUALS1 pad 1: /ROW0 -> unconnected-(KEQUALS1-Pad1)
- KEQUALS1 pad 2: /COL12 -> Net-(DEQUALS1-Pad2)
- KESC1 pad 2: /COL0 -> Net-(DESC1-Pad2)
- KF1 pad 2: /COL4 -> Net-(DF1-Pad2)
- KFIVE1 pad 2: /COL5 -> Net-(DFIVE1-Pad2)
- KFN1 pad 2: /COL11 -> Net-(DFN1-Pad2)
- KFOUR1 pad 2: /COL4 -> Net-(DFOUR1-Pad2)
- KFSLASH1 pad 2: /COL10 -> Net-(DFSLASH1-Pad2)
- KG1 pad 2: /COL5 -> Net-(DG1-Pad2)
- KH1 pad 2: /COL6 -> Net-(DH1-Pad2)
- KI1 pad 2: /COL8 -> Net-(DI1-Pad2)
- KJ1 pad 2: /COL7 -> Net-(DJ1-Pad2)
- KK1 pad 2: /COL8 -> Net-(DK1-Pad2)
- KL1 pad 2: /COL9 -> Net-(DL1-Pad2)
- KLALT1 pad 2: /COL2 -> Net-(DLALT1-Pad2)
- KLB1 pad 2: /COL11 -> Net-(DLB1-Pad2)
- KLCTRL1 pad 2: /COL0 -> Net-(DLCTRL1-Pad2)
- KLMETA1 pad 2: /COL1 -> Net-(DLMETA1-Pad2)
- KLS1 pad 2: /COL0 -> Net-(DLS1-Pad2)
- KM1 pad 2: /COL7 -> Net-(DM1-Pad2)
- KN1 pad 2: /COL6 -> Net-(DN1-Pad2)
- KNINE1 pad 2: /COL9 -> Net-(DNINE1-Pad2)
- KO1 pad 2: /COL9 -> Net-(DO1-Pad2)
- KONE1 pad 2: /COL1 -> Net-(DONE1-Pad2)
- KP1 pad 2: /COL10 -> Net-(DP1-Pad2)
- KPERIOD1 pad 2: /COL9 -> Net-(DPERIOD1-Pad2)
- KQ1 pad 2: /COL1 -> Net-(DQ1-Pad2)
- KR1 pad 2: /COL4 -> Net-(DR1-Pad2)
- KRALT1 pad 2: /COL8 -> Net-(DRALT1-Pad2)
- KRB1 pad 1: /ROW1 -> unconnected-(KRB1-Pad1)
- KRB1 pad 2: /COL12 -> Net-(DRB1-Pad2)
- KRCTRL1 pad 2: /COL10 -> Net-(DRCTRL1-Pad2)
- KRETURN1 pad 2: /COL12 -> Net-(DRETURN1-Pad2)
- KRMETA1 pad 2: /COL9 -> Net-(DRMETA1-Pad2)
- KRS1 pad 2: /COL11 -> Net-(DRS1-Pad2)
- KS1 pad 2: /COL2 -> Net-(DS1-Pad2)
- KSC1 pad 2: /COL10 -> Net-(DSC1-Pad2)
- KSEVEN1 pad 2: /COL7 -> Net-(DSEVEN1-Pad2)
- KSIX1 pad 2: /COL6 -> Net-(DSIX1-Pad2)
- KSPACE1 pad 2: /COL5 -> Net-(DSPACE1-Pad2)
- KT1 pad 2: /COL5 -> Net-(DT1-Pad2)
- KTAB1 pad 2: /COL0 -> Net-(DTAB1-Pad2)
- KTHREE1 pad 2: /COL3 -> Net-(DTHREE1-Pad2)
- KTWO1 pad 2: /COL2 -> Net-(DTWO1-Pad2)
- KU1 pad 2: /COL7 -> Net-(DU1-Pad2)
- KV1 pad 2: /COL4 -> Net-(DV1-Pad2)
- KW1 pad 2: /COL2 -> Net-(DW1-Pad2)
- KX1 pad 2: /COL2 -> Net-(DX1-Pad2)
- KY1 pad 2: /COL6 -> Net-(DY1-Pad2)
- KZ1 pad 2: /COL1 -> Net-(DZ1-Pad2)
- KZERO1 pad 2: /COL10 -> Net-(DZERO1-Pad2)
- M1 pad 1: unconnected-(U3-Pad1) -> DIN
- M1 pad 15: Net-(C1-Pad1) -> GND
- M1 pad 16: Net-(C3-Pad2) -> Net-(C3-Pad1)
- M1 pad 23: Net-(C1-Pad1) -> GND
- M1 pad 35: Net-(C1-Pad1) -> GND
- M1 pad 43: Net-(C1-Pad1) -> GND
- M1 pad 45: Net-(C1-Pad1) -> GND
- M1 pad 5: Net-(C1-Pad1) -> GND
- U1 pad A1/B12: Net-(C1-Pad1) -> GND
- U1 pad B1/A12: Net-(C1-Pad1) -> GND
- U2 pad 6: Net-(C1-Pad1) -> GND
- Y1 pad 1: Net-(C2-Pad2) -> Net-(C3-Pad1)
- Y1 pad 2: Net-(C1-Pad1) -> GND
- Y1 pad 3: Net-(C3-Pad2) -> Net-(C2-Pad2)
- Y1 pad 4: Net-(C1-Pad1) -> GND
Routing:
- net VCC: track 712.5 -> 0.00 mm, vias 7 -> 0
- net Net-(C1-Pad1): track 677.9 -> 0.00 mm, vias 4 -> 0
- net /ROW1: track 663.0 -> 0.00 mm, vias 4 -> 0
- net /ROW0: track 652.1 -> 0.00 mm, vias 2 -> 0
- net /ROW2: track 649.2 -> 0.00 mm, vias 2 -> 0
- net /ROW3: track 606.8 -> 0.00 mm, vias 4 -> 0
- net Net-(R2-Pad2): track 567.2 -> 0.00 mm, vias 1 -> 0
- net Net-(R1-Pad2): track 560.0 -> 0.00 mm, vias 1 -> 0
- net /ROW4: track 527.9 -> 0.00 mm, vias 4 -> 0
- net /COL11: track 298.6 -> 0.00 mm, vias 5 -> 0
- net /COL12: track 274.4 -> 0.00 mm, vias 4 -> 0
- net /COL13: track 267.8 -> 0.00 mm, vias 3 -> 0
- net /COL10: track 265.1 -> 0.00 mm, vias 5 -> 0
- net /COL9: track 242.4 -> 0.00 mm, vias 5 -> 0
- net /COL8: track 219.9 -> 0.00 mm, vias 5 -> 0
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Other:
- board size 289.8 x 99.2 mm -> 286 x 94.6 mm

Commit message: PCB design and schematic
Parts:
- moved C1 43.9 mm to (166.2, 99.2)
- moved R1 43.9 mm to (160.5, 96.0)
- moved R2 43.9 mm to (160.5, 93.9)
- moved Y1 39.6 mm to (162.5, 97.5)
- moved C2 31.1 mm to (159.9, 100.9)
- moved C3 27.5 mm to (156.0, 95.0)
- moved DG1 15.3 mm to (124.3, 61.6)
- moved DA1 15.3 mm to (48.1, 61.6)
- moved DAP1 15.3 mm to (238.6, 61.6)
- moved DB1 15.3 mm to (133.8, 80.7)
- moved DBSLASH1 15.3 mm to (276.7, 42.6)
- moved DBSPACE1 15.3 mm to (271.9, 23.5)
- moved DC1 15.3 mm to (95.7, 80.7)
- moved DCAPS1 15.3 mm to (21.9, 61.6)
- moved DCOMMA1 15.3 mm to (191.0, 80.7)
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Connections:
- KEQUALS1 pad 1: unconnected-(KEQUALS1-Pad1) -> /ROW0
- KRB1 pad 1: unconnected-(KRB1-Pad1) -> /ROW1
- M1 pad 10: /ROW2 -> Net-(M1-Pad10)
- M1 pad 11: /ROW1 -> Net-(M1-Pad11)
- M1 pad 12: /ROW0 -> unconnected-(M1-Pad12)
- M1 pad 18: /COL0 -> /ROW0
- M1 pad 19: /COL1 -> /ROW1
- M1 pad 20: /COL2 -> /ROW2
- M1 pad 21: /COL3 -> /ROW3
- M1 pad 22: /COL4 -> /ROW4
- M1 pad 25: /COL5 -> /COL0
- M1 pad 26: /COL6 -> /COL1
- M1 pad 27: /COL7 -> /COL2
- M1 pad 28: /COL8 -> /COL3
- M1 pad 29: /COL9 -> /COL4
- M1 pad 30: /COL10 -> /COL5
- M1 pad 31: /COL11 -> /COL6
- M1 pad 32: /COL12 -> /COL7
- M1 pad 33: /COL13 -> /COL8
- M1 pad 8: /ROW4 -> unconnected-(M1-Pad8)
- M1 pad 9: /ROW3 -> Net-(M1-Pad9)
- U2 pad 1: /ROW1 -> Net-(M1-Pad11)
- U2 pad 3: /ROW3 -> Net-(M1-Pad9)
- U2 pad 4: /ROW2 -> Net-(M1-Pad10)
Routing:
- net GND: track 0.00 -> 1374.7 mm
- net VCC: track 0.00 -> 1324.8 mm
- net /ROW0: track 0.00 -> 443.6 mm, vias 0 -> 4
- net /ROW1: track 0.00 -> 411.8 mm, vias 0 -> 2
- net /ROW2: track 0.00 -> 381.9 mm, vias 0 -> 2
- net /ROW3: track 0.00 -> 342.6 mm, vias 0 -> 2
- net /ROW4: track 0.00 -> 315.0 mm, vias 0 -> 2
- net Net-(LLS1-Pad4): track 0.00 -> 284.5 mm
- net Net-(LBSPACE1-Pad2): track 0.00 -> 281.5 mm, vias 0 -> 2
- net Net-(LBSLASH1-Pad2): track 0.00 -> 280.9 mm
- net Net-(LLCTRL1-Pad4): track 0.00 -> 276.2 mm
- net /COL8: track 0.00 -> 221.8 mm, vias 0 -> 8
- net /COL0: track 0.00 -> 192.6 mm, vias 0 -> 8
- net /COL7: track 0.00 -> 181.3 mm, vias 0 -> 7
- net /COL5: track 0.00 -> 170.9 mm, vias 0 -> 9
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Other:
- board size 286 x 94.6 mm -> 285 x 94.6 mm

Commit message: PCB done
Parts:
- moved Y1 53.3 mm to (109.5, 103.2), turned to 0 degrees
- moved C1 50.8 mm to (115.5, 96.5)
- moved U2 49.5 mm to (127.5, 98.2)
- moved R2 45.1 mm to (115.5, 91.0)
- moved R1 45.1 mm to (115.5, 93.8)
- moved C2 44.5 mm to (115.5, 104.0)
- moved C3 41.0 mm to (115.5, 101.2), turned to 180 degrees
Connections:
- M1 pad 36: unconnected-(M1-Pad36) -> /COL9
- M1 pad 37: unconnected-(M1-Pad37) -> /COL10
- M1 pad 38: unconnected-(M1-Pad38) -> /COL11
- M1 pad 39: unconnected-(M1-Pad39) -> /COL12
- M1 pad 40: unconnected-(M1-Pad40) -> /COL13
Routing:
- net /COL13: track 22.6 -> 232.3 mm, vias 2 -> 5
- net VCC: track 1324.8 -> 1528.5 mm, vias 0 -> 14
- net Net-(R1-Pad2): track 0.00 -> 194.6 mm, vias 0 -> 2
- net Net-(R2-Pad2): track 0.00 -> 192.4 mm, vias 0 -> 2
- net /COL12: track 53.2 -> 239.4 mm, vias 3 -> 6
- net DIN: track 0.00 -> 173.3 mm, vias 0 -> 2
- net /COL11: track 110.6 -> 268.8 mm, vias 5 -> 8
- net GND: track 1374.7 -> 1526.0 mm, vias 0 -> 11
- net /COL10: track 109.8 -> 252.4 mm, vias 5 -> 8
- net /COL9: track 104.1 -> 229.1 mm, vias 5 -> 8
- net Net-(M1-Pad10): track 0.00 -> 28.9 mm
- net Net-(M1-Pad13): track 0.00 -> 21.7 mm
- net Net-(M1-Pad9): track 0.00 -> 19.0 mm, vias 0 -> 2
- net Net-(M1-Pad11): track 0.00 -> 18.8 mm
- net Net-(C2-Pad2): track 0.00 -> 15.9 mm
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