File: design/pcb/USBKB.kicad_sch (KiCad schematic)
At the start: 192 parts, among them M1 ATMEGA32U4-MU, U1 USB4105-GF-A, U2 ICSP, Y1 Crystal_GND23

Commit message: PCB design and schematic
Connections:
- net COL0: now also M1.25 (PD4); no longer M1.18 (PD0)
- net COL1: now also M1.26 (PD6); no longer M1.19 (PD1)
- net COL10: no longer M1.30 (PB6)
- net COL11: no longer M1.31 (PC6)
- net COL12: no longer M1.32 (PC7)
- net COL13: no longer M1.33 (PE2)
- net COL2: now also M1.27 (PD7); no longer M1.20 (PD2)
- net COL3: now also M1.28 (PB4); no longer M1.21 (PD3)
- net COL4: now also M1.29 (PB5); no longer M1.22 (PD5)
- net COL5: now also M1.30 (PB6); no longer M1.25 (PD4)
- net COL6: now also M1.31 (PC6); no longer M1.26 (PD6)
- net COL7: now also M1.32 (PC7); no longer M1.27 (PD7)
- net COL8: now also M1.33 (PE2); no longer M1.28 (PB4)
- net COL9: no longer M1.29 (PB5)
- net ROW0: now also KEQUALS1.1, M1.18 (PD0); no longer M1.12 (PB7)
- net ROW1: now also KRB1.1, M1.19 (PD1); no longer M1.11 (PB3(MISO)), U2.1 (MISO)
- net ROW2: now also M1.20 (PD2); no longer M1.10 (PB2(MOSI)), U2.4 (MOSI)
- net ROW3: now also M1.21 (PD3); no longer M1.9 (PB1(SCL)), U2.3 (SCK)
- net ROW4: now also M1.22 (PD5); no longer M1.8 (PB0(SS))
- new net: M1.10 (PB2(MOSI)), U2.4 (MOSI)
- new net: M1.11 (PB3(MISO)), U2.1 (MISO)
- new net: M1.9 (PB1(SCL)), U2.3 (SCK)
Changed lines of the file:
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@@
   (junction (at 360.68 129.54) (diameter 0) (color 0 0 0 0)
   )
+  (junction (at 241.3 34.29) (diameter 0) (color 0 0 0 0)
+  )
   (junction (at 73.66 52.07) (diameter 0) (color 0 0 0 0)
   )
@@
   (junction (at 289.56 154.94) (diameter 0) (color 0 0 0 0)
   )
+  (junction (at 241.3 22.86) (diameter 0) (color 0 0 0 0)
+  )
   (junction (at 287.02 185.42) (diameter 0) (color 0 0 0 0)
   )
@@
     (stroke (width 0) (type default) (color 0 0 0 0))
   )
+  (wire (pts (xy 241.3 22.86) (xy 259.08 22.86))
+    (stroke (width 0) (type default) (color 0 0 0 0))
+  )
   (wire (pts (xy 233.68 52.07) (xy 234.95 52.07))
     (stroke (width 0) (type default) (color 0 0 0 0))
@@
     (stroke (width 0) (type default) (color 0 0 0 0))
   )
+  (wire (pts (xy 241.3 21.59) (xy 241.3 22.86))
+    (stroke (width 0) (type default) (color 0 0 0 0))
+  )
   (wire (pts (xy 73.66 128.27) (xy 73.66 167.64))
     (stroke (width 0) (type default) (color 0 0 0 0))
@@
     (stroke (width 0) (type default) (color 0 0 0 0))
   )
-  (wire (pts (xy 223.52 22.86) (xy 259.08 22.86))
+  (wire (pts (xy 223.52 22.86) (xy 241.3 22.86))
     (stroke (width 0) (type default) (color 0 0 0 0))
   )
@@
     (stroke (width 0) (type default) (color 0 0 0 0))
   )
+  (wire (pts (xy 241.3 33.02) (xy 241.3 34.29))
+    (stroke (width 0) (type default) (color 0 0 0 0))
+  )
   (wire (pts (xy 55.88 40.64) (xy 55.88 52.07))
     (stroke (width 0) (type default) (color 0 0 0 0))
@@
     (stroke (width 0) (type default) (color 0 0 0 0))
   )
-  (wire (pts (xy 223.52 34.29) (xy 259.08 34.29))
+  (wire (pts (xy 223.52 34.29) (xy 241.3 34.29))
     (stroke (width 0) (type default) (color 0 0 0 0))
   )
@@
     (stroke (width 0) (type default) (color 0 0 0 0))
   )
+  (wire (pts (xy 241.3 34.29) (xy 259.08 34.29))
+    (stroke (width 0) (type default) (color 0 0 0 0))
+  )
   (wire (pts (xy 252.73 226.06) (xy 252.73 220.98))
     (stroke (width 0) (type default) (color 0 0 0 0))
@@
     (stroke (width 0) (type default) (color 0 0 0 0))
   )
-  (label "COL0" (at 128.27 167.64 180)
-    (effects (font (size 1.27 1.27)) (justify right bottom))
-  )
-  (label "ROW2" (at 128.27 132.08 180)
+  (label "COL5" (at 128.27 142.24 180)
     (effects (font (size 1.27 1.27)) (justify right bottom))
   )
@@
     (effects (font (size 1.27 1.27)) (justify left bottom))
   )
-  (label "COL5" (at 128.27 177.8 180)
+  (label "ROW4" (at 128.27 180.34 180)
     (effects (font (size 1.27 1.27)) (justify right bottom))
   )
-  (label "COL11" (at 128.27 121.92 180)
-    (effects (font (size 1.27 1.27)) (justify right bottom))
+  (label "COL11" (at 234.95 81.28 90)
+    (effects (font (size 1.27 1.27)) (justify left bottom))
   )
-  (label "COL3" (at 128.27 175.26 180)
+  (label "ROW0" (at 128.27 167.64 180)
     (effects (font (size 1.27 1.27)) (justify right bottom))
   )
-  (label "COL11" (at 234.95 81.28 90)
-    (effects (font (size 1.27 1.27)) (justify left bottom))
+  (label "COL8" (at 128.27 114.3 180)
+    (effects (font (size 1.27 1.27)) (justify right bottom))
   )
   (label "COL7" (at 162.56 81.28 90)
@@
     (effects (font (size 1.27 1.27)) (justify left bottom))
   )
-  (label "COL6" (at 128.27 182.88 180)
+  (label "COL9" (at 127 212.09 180)
+    (effects (font (size 1.27 1.27)) (justify right bottom))
+  )
+  (label "COL11" (at 127 217.17 180)
+    (effects (font (size 1.27 1.27)) (justify right bottom))
+  )
+  (label "COL10" (at 128.27 214.63 180)
     (effects (font (size 1.27 1.27)) (justify right bottom))
   )
-  (label "COL1" (at 128.27 170.18 180)
+  (label "ROW2" (at 128.27 172.72 180)
     (effects (font (size 1.27 1.27)) (justify right bottom))
   )
@@
     (effects (font (size 1.27 1.27)) (justify left bottom))
   )
-  (label "COL4" (at 128.27 180.34 180)
+  (label "COL4" (at 128.27 139.7 180)
     (effects (font (size 1.27 1.27)) (justify right bottom))
   )
@@
     (effects (font (size 1.27 1.27)) (justify left bottom))
   )
-  (label "COL2" (at 128.27 172.72 180)
-    (effects (font (size 1.27 1.27)) (justify right bottom))
+  (label "COL12" (at 252.73 81.28 90)
+    (effects (font (size 1.27 1.27)) (justify left bottom))
   )
-  (label "COL7" (at 128.27 185.42 180)
+  (label "COL13" (at 127 226.06 180)
     (effects (font (size 1.27 1.27)) (justify right bottom))
   )
-  (label "COL13" (at 128.27 114.3 180)
+  (label "COL12" (at 127 220.98 180)
     (effects (font (size 1.27 1.27)) (justify right bottom))
   )
-  (label "COL12" (at 252.73 81.28 90)
-    (effects (font (size 1.27 1.27)) (justify left bottom))
+  (label "COL7" (at 128.27 119.38 180)
+    (effects (font (size 1.27 1.27)) (justify right bottom))
   )
   (label "COL8" (at 180.34 81.28 90)
     (effects (font (size 1.27 1.27)) (justify left bottom))
   )
-  (label "ROW3" (at 128.27 129.54 180)
-    (effects (font (size 1.27 1.27)) (justify right bottom))
-  )
-  (label "COL10" (at 128.27 142.24 180)
+  (label "COL0" (at 128.27 177.8 180)
     (effects (font (size 1.27 1.27)) (justify right bottom))
   )
@@
     (effects (font (size 1.27 1.27)) (justify left bottom))
   )
-  (label "COL6" (at 144.78 81.28 90)
-    (effects (font (size 1.27 1.27)) (justify left bottom))
-  )
-  (label "COL9" (at 128.27 139.7 180)
-    (effects (font (size 1.27 1.27)) (justify right bottom))
-  )
-  (label "COL8" (at 128.27 137.16 180)
+  (label "ROW1" (at 128.27 170.18 180)
     (effects (font (size 1.27 1.27)) (justify right bottom))
   )
-  (label "COL12" (at 128.27 119.38 180)
-    (effects (font (size 1.27 1.27)) (justify right bottom))
+  (label "COL6" (at 144.78 81.28 90)
+    (effects (font (size 1.27 1.27)) (justify left bottom))
   )
-  (label "ROW1" (at 128.27 134.62 180)
+  (label "COL3" (at 128.27 137.16 180)
     (effects (font (size 1.27 1.27)) (justify right bottom))
   )
-  (label "ROW4" (at 128.27 127 180)
+  (label "COL1" (at 128.27 182.88 180)
     (effects (font (size 1.27 1.27)) (justify right bottom))
   )
-  (label "ROW0" (at 128.27 144.78 180)
+  (label "COL6" (at 128.27 121.92 180)
     (effects (font (size 1.27 1.27)) (justify right bottom))
   )
@@
     (effects (font (size 1.27 1.27)) (justify left bottom))
   )
+  (label "ROW3" (at 128.27 175.26 180)
+    (effects (font (size 1.27 1.27)) (justify right bottom))
+  )
   (label "COL5" (at 127 81.28 90)
     (effects (font (size 1.27 1.27)) (justify left bottom))
   )
+  (label "COL2" (at 128.27 185.42 180)
+    (effects (font (size 1.27 1.27)) (justify right bottom))
+  )
   (label "ROW0" (at 19.05 22.86 0)

Commit message: PCB done
Connections:
- net COL10: now also M1.37 (PF6)
- net COL11: now also M1.38 (PF5)
- net COL12: now also M1.39 (PF4)
- net COL13: now also M1.40 (PF1)
- net COL9: now also M1.36 (PF7)
- no-connect marks 11 -> 8
Changed lines of the file:
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@@
   (junction (at 38.1 74.93) (diameter 0) (color 0 0 0 0)
   )
-  (no_connect (at 121.92 162.56))
   (no_connect (at 121.92 149.86))
-  (no_connect (at 121.92 152.4))
-  (no_connect (at 121.92 160.02))
-  (no_connect (at 121.92 157.48))
-  (no_connect (at 121.92 154.94))
   (no_connect (at 358.14 226.06))
   (no_connect (at 27.94 115.57))
@@
   (no_connect (at 27.94 130.81))
   (no_connect (at 27.94 133.35))
+  (no_connect (at 121.92 127))
+  (no_connect (at 121.92 144.78))
   (wire (pts (xy 121.92 114.3) (xy 128.27 114.3))
     (stroke (width 0) (type default) (color 0 0 0 0))
@@
     (stroke (width 0) (type default) (color 0 0 0 0))
   )
+  (wire (pts (xy 121.92 162.56) (xy 128.27 162.56))
+    (stroke (width 0) (type default) (color 0 0 0 0))
+  )
   (wire (pts (xy 64.77 196.85) (xy 133.35 196.85))
     (stroke (width 0) (type default) (color 0 0 0 0))
@@
     (stroke (width 0) (type default) (color 0 0 0 0))
   )
-  (wire (pts (xy 121.92 127) (xy 128.27 127))
-    (stroke (width 0) (type default) (color 0 0 0 0))
-  )
   (wire (pts (xy 87.63 33.02) (xy 90.17 33.02))
     (stroke (width 0) (type default) (color 0 0 0 0))
@@
     (stroke (width 0) (type default) (color 0 0 0 0))
   )
+  (wire (pts (xy 121.92 160.02) (xy 128.27 160.02))
+    (stroke (width 0) (type default) (color 0 0 0 0))
+  )
   (wire (pts (xy 342.9 124.46) (xy 342.9 129.54))
     (stroke (width 0) (type default) (color 0 0 0 0))
@@
     (stroke (width 0) (type default) (color 0 0 0 0))
   )
+  (wire (pts (xy 121.92 157.48) (xy 128.27 157.48))
+    (stroke (width 0) (type default) (color 0 0 0 0))
+  )
   (wire (pts (xy 73.66 175.26) (xy 78.74 175.26))
     (stroke (width 0) (type default) (color 0 0 0 0))
@@
     (stroke (width 0) (type default) (color 0 0 0 0))
   )
-  (wire (pts (xy 121.92 144.78) (xy 128.27 144.78))
-    (stroke (width 0) (type default) (color 0 0 0 0))
-  )
   (wire (pts (xy 38.1 74.93) (xy 38.1 81.28))
     (stroke (width 0) (type default) (color 0 0 0 0))
@@
     (stroke (width 0) (type default) (color 0 0 0 0))
   )
+  (wire (pts (xy 121.92 154.94) (xy 128.27 154.94))
+    (stroke (width 0) (type default) (color 0 0 0 0))
+  )
   (wire (pts (xy 180.34 74.93) (xy 180.34 81.28))
     (stroke (width 0) (type default) (color 0 0 0 0))
@@
   )
   (wire (pts (xy 147.32 226.06) (xy 147.32 231.14))
+    (stroke (width 0) (type default) (color 0 0 0 0))
+  )
+  (wire (pts (xy 121.92 152.4) (xy 128.27 152.4))
     (stroke (width 0) (type default) (color 0 0 0 0))
   )
@@
     (effects (font (size 1.27 1.27)) (justify left bottom))
   )
-  (label "COL9" (at 127 212.09 180)
+  (label "COL11" (at 128.27 157.48 180)
     (effects (font (size 1.27 1.27)) (justify right bottom))
   )
-  (label "COL11" (at 127 217.17 180)
-    (effects (font (size 1.27 1.27)) (justify right bottom))
-  )
-  (label "COL10" (at 128.27 214.63 180)
+  (label "COL10" (at 128.27 160.02 180)
     (effects (font (size 1.27 1.27)) (justify right bottom))
   )
@@
     (effects (font (size 1.27 1.27)) (justify left bottom))
   )
-  (label "COL13" (at 127 226.06 180)
+  (label "COL13" (at 128.27 152.4 180)
     (effects (font (size 1.27 1.27)) (justify right bottom))
   )
-  (label "COL12" (at 127 220.98 180)
+  (label "COL12" (at 128.27 154.94 180)
     (effects (font (size 1.27 1.27)) (justify right bottom))
   )
@@
     (effects (font (size 1.27 1.27)) (justify right bottom))
   )
+  (label "COL9" (at 128.27 162.56 180)
+    (effects (font (size 1.27 1.27)) (justify right bottom))
+  )
